File: HW/Multislope 3I.kicad_pcb (KiCad board)
At the start: 4 copper layers, 100 x 74 mm, 126 parts, among them J1 INT, J10 PWR, J11 TEST, J12 UART, J13 INPUT, J14 SLOPE, J15 PWR, J2 TEST, J3 COMP, J4 SLOT, J5 SLOT, J6 SLOT, J7 SLOPE2, J8 PWR, J9 SLOT, SW1 RST, U1 OPA21xx, U10 LM311, U11 NE5534, U12 OPA197, U14 431, U15 MCP3202, U16 Pico, U17 LM35, U18 ADuM121N, U2 LM399, U20 HT7533, U21 HT7550, U3 CD4053B, U4 OPA1xx, U5 OPA1xx, U6 OPA1xx, U7 431, U8 431, U9 408

Commit message: Reference startup circuit added
Parts:
- added D3: 4148, Diode_SMD:D_SOD-323, F.Cu at (96.8, 98.4)
- added R43: 100K, Resistor_SMD:R_0603_1608Metric, F.Cu at (97.2, 105.4)
- R6, R7: value 0R -> 3K1
Connections:
- R6 pad 2: /+REF -> Net-(R6-Pad2)
Routing:
- net +15V: track 290.4 -> 296.3 mm, vias 24 -> 25
- net /+REF: track 116.8 -> 113.0 mm
- net /RAW: track 97.5 -> 101.2 mm
- net Net-(R6-Pad2): track 0.00 -> 1.71 mm
