File: HW/Multislope 3I.kicad_pcb (KiCad board)
At the start: 4 copper layers, 100 x 74 mm, 128 parts, among them J1 INT, J10 PWR, J11 TEST, J12 UART, J13 INPUT, J14 SLOPE, J15 PWR, J2 TEST, J3 COMP, J4 SLOT, J5 SLOT, J6 SLOT, J7 SLOPE2, J8 PWR, J9 SLOT, SW1 RST, U1 OPA21xx, U10 LM311, U11 NE5534, U12 OPA197, U14 431, U15 MCP3202, U16 Pico, U17 LM35, U18 ADuM121N, U2 LM399, U20 HT7533, U21 HT7550, U3 CD4053B, U4 OPA1xx, U5 OPA1xx, U6 OPA1xx, U7 431, U8 431, U9 408

Commit message: added files
Parts:
- U3: value CD4053B -> SN74LV4053
Connections:
- J2 pad 5: Net-(J2-Pad5) -> /PWMA
- J2 pad 6: Net-(J2-Pad6) -> /PWMB
- J2 pad 7: Net-(J2-Pad7) -> /MEAS
- R27 pad 2: Net-(J2-Pad5) -> /PWMA
- R28 pad 2: Net-(J2-Pad6) -> /PWMB
- R29 pad 2: Net-(J2-Pad7) -> /MEAS
- U16 pad 5: Net-(J2-Pad5) -> /PWMA
- U16 pad 6: Net-(J2-Pad6) -> /PWMB
- U16 pad 7: Net-(J2-Pad7) -> /MEAS
Routing:
- net /PWMA: track 37.1 -> 59.6 mm
- net Net-(J2-Pad5): track 22.5 -> 0.00 mm
- net /PWMB: track 35.0 -> 56.9 mm
- net Net-(J2-Pad6): track 21.9 -> 0.00 mm
- net Net-(J2-Pad7): track 21.4 -> 0.00 mm
- net /MEAS: track 32.8 -> 54.2 mm
